File: SDcore/SDcore.kicad_pcb (KiCad board)
At the start: 4 copper layers, 24 x 32 mm, 38 parts, among them J1 SD_Card_Device, Q1 L2N7002WT1G, U1 RP2350A_C42411118, U2 NMUX27518EPWJ, U3 W25Q128JVEIQ_TR, X1 ABM8-272-T3_C20625731

Commit message: Updated schematics and PCB, rewired some GPIOs
Connections:
- GPIO1 pad 23: GND -> P_GPIO_2
- U1 pad 2: GPIO_0 -> DATA_DIRECT_1
- U1 pad 3: DATA_DIRECT_1 -> DATA_DIRECT_2
- U1 pad 4: DATA_DIRECT_2 -> P_GPIO_2
Routing:
- net P_GPIO_2: track 0.00 -> 32.2 mm, vias 0 -> 4
- net GND: track 168.3 -> 158.2 mm, vias 45 -> 44
