File: SDcore/SDcore.kicad_sch (KiCad schematic)
At the start: 39 parts, among them J1 SD_Card_Device, Q1 L2N7002WT1G, U1 RP2350A_C42411118, U2 NMUX27518EPWJ, U3 W25Q128JVEIQ_TR, X1 ABM8-272-T3_C20625731

Commit message: Updated schematics and PCB, rewired some GPIOs
Connections:
- net GPIO_0 is gone; now on net DATA_DIRECT_1: U1.2 (GPIO0)
- net DATA_DIRECT_1: no longer U1.3 (GPIO1)
- net DATA_DIRECT_2: now also U1.3 (GPIO1); no longer U1.4 (GPIO2)
- net GND: no longer GPIO1.23
- new net P_GPIO_2: GPIO1.23, U1.4 (GPIO2)
Changed lines of the file:
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@@
 	)
 	(junction
-		(at 139.7 25.4)
-		(diameter 0)
-		(color 0 0 0 0)
-	)
-	(junction
 		(at 29.21 62.23)
 		(diameter 0)
@@
 	(wire
 		(pts
-			(xy 139.7 25.4) (xy 137.16 25.4)
-		)
-		(stroke
-			(width 0)
-			(type default)
-		)
-	)
-	(wire
-		(pts
 			(xy 160.02 106.68) (xy 142.24 106.68)
 		)
@@
 		)
 	)
+	(global_label "P_GPIO_2"
+		(shape input)
+		(at 196.85 63.5 180)
+		(fields_autoplaced yes)
+		(effects
+			(font
+				(size 1.27 1.27)
+			)
+			(justify right)
+		)
+		(property "Intersheetrefs" "${INTERSHEET_REFS}"
+			(at 184.9748 63.5 0)
+			(effects
+				(font
+					(size 1.27 1.27)
+				)
+				(justify right)
+				(hide yes)
+			)
+		)
+	)
 	(global_label "IN_CMD"
 		(shape input)
@@
 		)
 	)
+	(global_label "DATA_DIRECT_1"
+		(shape input)
+		(at 101.6 130.81 180)
+		(fields_autoplaced yes)
+		(effects
+			(font
+				(size 1.27 1.27)
+			)
+			(justify right)
+		)
+		(property "Intersheetrefs" "${INTERSHEET_REFS}"
+			(at 84.5239 130.81 0)
+			(effects
+				(font
+					(size 1.27 1.27)
+				)
+				(justify right)
+				(hide yes)
+			)
+		)
+	)
 	(global_label "IN_DAT1"
 		(shape input)
@@
 		)
 	)
-	(global_label "DATA_DIRECT_1"
+	(global_label "DATA_DIRECT_2"
 		(shape input)
 		(at 101.6 133.35 180)
@@
 	(global_label "BOOT_SIGNAL"
 		(shape input)
-		(at 137.16 25.4 180)
+		(at 139.7 25.4 180)
 		(fields_autoplaced yes)
 		(effects
@@
 		)
 		(property "Intersheetrefs" "${INTERSHEET_REFS}"
-			(at 121.7771 25.4 0)
+			(at 124.3171 25.4 0)
 			(effects
 				(font
@@
 		)
 	)
-	(global_label "GPIO_0"
-		(shape input)
-		(at 101.6 130.81 180)
-		(fields_autoplaced yes)
-		(effects
-			(font
-				(size 1.27 1.27)
-			)
-			(justify right)
-		)
-		(property "Intersheetrefs" "${INTERSHEET_REFS}"
-			(at 91.9624 130.81 0)
-			(effects
-				(font
-					(size 1.27 1.27)
-				)
-				(justify right)
-				(hide yes)
-			)
-		)
-	)
 	(global_label "SPI1_SCK_CLK"
 		(shape input)
@@
 		)
 	)
-	(global_label "DATA_DIRECT_2"
-		(shape input)
-		(at 101.6 135.89 180)
-		(fields_autoplaced yes)
-		(effects
-			(font
-				(size 1.27 1.27)
-			)
-			(justify right)
-		)
-		(property "Intersheetrefs" "${INTERSHEET_REFS}"
-			(at 84.5239 135.89 0)
-			(effects
-				(font
-					(size 1.27 1.27)
-				)
-				(justify right)
-				(hide yes)
-			)
-		)
-	)
 	(global_label "P_GPIO20"
 		(shape input)
@@
 		)
 	)
+	(global_label "P_GPIO_2"
+		(shape input)
+		(at 101.6 135.89 180)
+		(fields_autoplaced yes)
+		(effects
+			(font
+				(size 1.27 1.27)
+			)
+			(justify right)
+		)
+		(property "Intersheetrefs" "${INTERSHEET_REFS}"
+			(at 89.7248 135.89 0)
+			(effects
+				(font
+					(size 1.27 1.27)
+				)
+				(justify right)
+				(hide yes)
+			)
+		)
+	)
 	(global_label "P_GPIO20"
 		(shape input)
@@
 					(unit 1)
 				)
-			)
-		)
-	)
-	(symbol
-		(lib_id "power:GND")
-		(at 196.85 63.5 270)
-		(unit 1)
-		(exclude_from_sim no)
-		(in_bom yes)
-		(on_board yes)
-		(dnp no)
-		(fields_autoplaced yes)
-		(property "Reference" "#PWR045"
-			(at 190.5 63.5 0)
-			(effects
-				(font
-					(size 1.27 1.27)
-				)
-				(hide yes)
-			)
-		)
-		(property "Value" "GND"
-			(at 193.04 63.4999 90)
-			(effects
-				(font
-					(size 1.27 1.27)
-				)
-				(justify right)
-			)
-		)
-		(property "Footprint" ""
-			(at 196.85 63.5 0)
-			(effects
-				(font
-					(size 1.27 1.27)
-				)
-				(hide yes)
-			)
-		)
-		(property "Datasheet" ""
-			(at 196.85 63.5 0)
-			(effects
-				(font
-					(size 1.27 1.27)
-				)
-				(hide yes)
-			)
-		)
-		(property "Description" "Power symbol creates a global label with name \"GND\" , ground"
-			(at 196.85 63.5 0)
-			(effects
-				(font
-					(size 1.27 1.27)
-				)
-				(hide yes)
-			)
-		)
-		(pin "1"
-		)
-		(instances
-			(project "SDcore"
-				(path "/4923730a-c063-43f4-b067-8ce717e5d6d0"
-					(reference "#PWR045")
-					(unit 1)
-				)

Commit message: Added pull-up resistors to the micro-SD card slot
Parts:
- removed R12: 4.7k, JLCImport:CRCW04024K70FKEDC, symbol JLCImport:CRCW04024K70FKEDC
- added R11, R12, R13, R14, R15, R16: 10k, JLCImport:CRCW040210K0FKED, symbol JLCImport:CRCW040210K0FKED
- renumbered R11 to R7
Connections:
- net +3V3: now also R11.2, R12.2, R13.2, R14.2, R15.2, R16.2
- net DATA_SD_SNIFF_1: now also R16.1
- net DATA_SD_SNIFF_2: now also R11.1
- net OUT_CLK: now also R14.1
- net OUT_CMD: now also R13.1
- net OUT_DAT0: now also R15.1
- net OUT_DAT3: now also R12.1
Other:
- moved on the sheet: LED1, LED2, LED3, R10, R8, R9, U2

Commit message: I forgot that traces have clearances too, so I added them; Added test pads for reset and bootsel functions; Removed ground zone underneath MCU to reduce potential interference.
Parts:
- added TP1: TestPoint_Alt, TestPoint:TestPoint_Pad_1.0x1.0mm, symbol Connector:TestPoint_Alt
- added TP2, TP3: TestPoint, TestPoint:TestPoint_Pad_D1.0mm, symbol Connector:TestPoint
Connections:
- net BOOT_SIGNAL: now also TP2.1
- net GND: now also TP1.1
- net RUN: now also TP3.1
